Commit message: Update with current state

File: urdf/assembly_2.urdf (robot description, URDF)
Before this commit: robot assembly_2, 326 links, 325 joints
Links:
- added link water_tank, mass 0.0001; collision mesh filename=package://assembly_2/meshes/water_tank.stl scale=1 1 1; visual mesh filename=package://assembly_2/meshes/water_tank.stl scale=1 1 1
- added link water_tank_2, mass 1e-05; collision cylinder length=0.045 radius=0.01125; visual cylinder length=0.045 radius=0.01125
Joints:
- added joint water_tank_2_joint: type fixed, parent part_1_48, child water_tank_2, origin xyz=0 0 0.0225 rpy=0 0 0
- added joint water_tank_joint: type fixed, parent root, child water_tank, origin xyz=-0.252742 0.361599 -0.481520 rpy=-1.5708 0 0
- joint revolute_1: type continuous -> fixed
- joint revolute_2: type continuous -> fixed
- joint revolute_3: axis -1 0 0 -> 1 0 0
- joint revolute_4: axis -1 -0 -0 -> 1 0 0
