Commit message: Update with current state

File: new_robot/urdf/new_robot copy.urdf (robot description, URDF)
Before this commit: robot new_robot, 70 links, 69 joints
Links:
- link default: mass 0.000267863 -> 0.015
- link default_1: mass 0.000267863 -> 0.015
- link default_10: mass 0.000267863 -> 0.015
- link default_11: mass 0.000267863 -> 0.015
- link default_12: mass 0.000267863 -> 0.015
- link default_13: mass 0.000267863 -> 0.015
- link default_2: mass 0.000267863 -> 0.015
- link default_3: mass 0.000267863 -> 0.015
- link default_4: mass 0.000267863 -> 0.015
- link default_5: mass 0.000267863 -> 0.015
- link default_6: mass 0.000267863 -> 0.015
- link default_7: mass 0.000267863 -> 0.015
- link default_8: mass 0.000267863 -> 0.015
- link default_9: mass 0.000267863 -> 0.015
- link part_1_1: mass 2.44526e-05 -> 0.15
- link part_1_12: mass 2.44526e-05 -> 0.15
- link part_1_13: mass 2.44526e-05 -> 0.15
- link part_1_9: mass 2.44526e-05 -> 0.15
