Commit message: Update with current state

File: new_robot/urdf/new_robot.urdf (robot description, URDF)
Before this commit: robot new_robot, 69 links, 68 joints
Links:
- link bjj02040274_gl60ii_Å_à_Ç_1_solid1: geometry collision mesh filename=package://new_robot/meshes/BJJ02040274_GL60II_______1_solid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 scale=1 1 1; visual mesh filename=package://new_robot/meshes/BJJ02040274_GL60II_______1_solid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 scale=1 1 1
- link bjj02040274_gl60ii_Å_à_Ç_1_solid1_1: geometry collision mesh filename=package://new_robot/meshes/BJJ02040274_GL60II_______1_solid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 scale=1 1 1; visual mesh filename=package://new_robot/meshes/BJJ02040274_GL60II_______1_solid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 scale=1 1 1
- link body2: geometry collision mesh filename=package://new_robot/meshes/Body2.stl scale=1 1 1; visual mesh filename=package://new_robot/meshes/Body2.stl scale=1 1 1
- link body2_1: geometry collision mesh filename=package://new_robot/meshes/Body2.stl scale=1 1 1; visual mesh filename=package://new_robot/meshes/Body2.stl scale=1 1 1
- link body2_2: geometry collision mesh filename=package://new_robot/meshes/Body2.stl scale=1 1 1; visual mesh filename=package://new_robot/meshes/Body2.stl scale=1 1 1
- link body2_3: geometry collision mesh filename=package://new_robot/meshes/Body2.stl scale=1 1 1; visual mesh filename=package://new_robot/meshes/Body2.stl scale=1 1 1
- link default: geometry collision mesh filename=package://new_robot/meshes/Default.stl scale=1 1 1; visual mesh filename=package://new_robot/meshes/Default.stl scale=1 1 1
- link default_1: geometry collision mesh filename=package://new_robot/meshes/Default.stl scale=1 1 1; visual mesh filename=package://new_robot/meshes/Default.stl scale=1 1 1
- link default_10: geometry collision mesh filename=package://new_robot/meshes/Default.stl scale=1 1 1; visual mesh filename=package://new_robot/meshes/Default.stl scale=1 1 1
- link default_11: geometry collision mesh filename=package://new_robot/meshes/Default.stl scale=1 1 1; visual mesh filename=package://new_robot/meshes/Default.stl scale=1 1 1
- link default_12: geometry collision mesh filename=package://new_robot/meshes/Default.stl scale=1 1 1; visual mesh filename=package://new_robot/meshes/Default.stl scale=1 1 1
- link default_13: geometry collision mesh filename=package://new_robot/meshes/Default.stl scale=1 1 1; visual mesh filename=package://new_robot/meshes/Default.stl scale=1 1 1
- link default_2: geometry collision mesh filename=package://new_robot/meshes/Default.stl scale=1 1 1; visual mesh filename=package://new_robot/meshes/Default.stl scale=1 1 1
- link default_3: geometry collision mesh filename=package://new_robot/meshes/Default.stl scale=1 1 1; visual mesh filename=package://new_robot/meshes/Default.stl scale=1 1 1
- link default_4: geometry collision mesh filename=package://new_robot/meshes/Default.stl scale=1 1 1; visual mesh filename=package://new_robot/meshes/Default.stl scale=1 1 1
- link default_5: geometry collision mesh filename=package://new_robot/meshes/Default.stl scale=1 1 1; visual mesh filename=package://new_robot/meshes/Default.stl scale=1 1 1
- link default_6: geometry collision mesh filename=package://new_robot/meshes/Default.stl scale=1 1 1; visual mesh filename=package://new_robot/meshes/Default.stl scale=1 1 1
- link default_7: geometry collision mesh filename=package://new_robot/meshes/Default.stl scale=1 1 1; visual mesh filename=package://new_robot/meshes/Default.stl scale=1 1 1
- link default_8: geometry collision mesh filename=package://new_robot/meshes/Default.stl scale=1 1 1; visual mesh filename=package://new_robot/meshes/Default.stl scale=1 1 1
- link default_9: geometry collision mesh filename=package://new_robot/meshes/Default.stl scale=1 1 1; visual mesh filename=package://new_robot/meshes/Default.stl scale=1 1 1
- link gb_fastener_screws_hshcs_m3x5_s_1_solid1: geometry collision mesh filename=package://new_robot/meshes/GB_FASTENER_SCREWS_HSHCS_M3X5_S_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 scale=1 1 1; visual mesh filename=package://new_robot/meshes/GB_FASTENER_SCREWS_HSHCS_M3X5_S_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 scale=1 1 1
- link gb_fastener_screws_hshcs_m3x5_s_1_solid1_1: geometry collision mesh filename=package://new_robot/meshes/GB_FASTENER_SCREWS_HSHCS_M3X5_S_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 scale=1 1 1; visual mesh filename=package://new_robot/meshes/GB_FASTENER_SCREWS_HSHCS_M3X5_S_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 scale=1 1 1
- link gb_fastener_screws_hshcs_m3x5_s_2_solid1: geometry collision mesh filename=package://new_robot/meshes/GB_FASTENER_SCREWS_HSHCS_M3X5_S_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 scale=1 1 1; visual mesh filename=package://new_robot/meshes/GB_FASTENER_SCREWS_HSHCS_M3X5_S_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 scale=1 1 1
- link gb_fastener_screws_hshcs_m3x5_s_2_solid1_1: geometry collision mesh filename=package://new_robot/meshes/GB_FASTENER_SCREWS_HSHCS_M3X5_S_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 scale=1 1 1; visual mesh filename=package://new_robot/meshes/GB_FASTENER_SCREWS_HSHCS_M3X5_S_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 scale=1 1 1
- link gb_fastener_screws_hshcs_m3x5_s_4_solid1: geometry collision mesh filename=package://new_robot/meshes/GB_FASTENER_SCREWS_HSHCS_M3X5_S_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 scale=1 1 1; visual mesh filename=package://new_robot/meshes/GB_FASTENER_SCREWS_HSHCS_M3X5_S_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 scale=1 1 1
- link gb_fastener_screws_hshcs_m3x5_s_4_solid1_1: geometry collision mesh filename=package://new_robot/meshes/GB_FASTENER_SCREWS_HSHCS_M3X5_S_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 scale=1 1 1; visual mesh filename=package://new_robot/meshes/GB_FASTENER_SCREWS_HSHCS_M3X5_S_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 scale=1 1 1
- link gl60_v1_0_240806a_1_solid86: geometry collision mesh filename=package://new_robot/meshes/GL60_V1_0_240806A_1_solid86.stl scale=1 1 1; visual mesh filename=package://new_robot/meshes/GL60_V1_0_240806A_1_solid86.stl scale=1 1 1
- link gl60_v1_0_240806a_1_solid86_1: geometry collision mesh filename=package://new_robot/meshes/GL60_V1_0_240806A_1_solid86.stl scale=1 1 1; visual mesh filename=package://new_robot/meshes/GL60_V1_0_240806A_1_solid86.stl scale=1 1 1
- link gl60_v1_0_240806a_1_solid87: geometry collision mesh filename=package://new_robot/meshes/GL60_V1_0_240806A_1_solid87.stl scale=1 1 1; visual mesh filename=package://new_robot/meshes/GL60_V1_0_240806A_1_solid87.stl scale=1 1 1
- link gl60_v1_0_240806a_1_solid87_1: geometry collision mesh filename=package://new_robot/meshes/GL60_V1_0_240806A_1_solid87.stl scale=1 1 1; visual mesh filename=package://new_robot/meshes/GL60_V1_0_240806A_1_solid87.stl scale=1 1 1
- link m3_ÂÝÎÆ__1: geometry collision mesh filename=package://new_robot/meshes/M3_______1.stl scale=1 1 1; visual mesh filename=package://new_robot/meshes/M3_______1.stl scale=1 1 1
- link m3_ÂÝÎÆ__1_1: geometry collision mesh filename=package://new_robot/meshes/M3_______1.stl scale=1 1 1; visual mesh filename=package://new_robot/meshes/M3_______1.stl scale=1 1 1
- link none: geometry collision mesh filename=package://new_robot/meshes/NONE.stl scale=1 1 1; visual mesh filename=package://new_robot/meshes/NONE.stl scale=1 1 1
- link none_1: geometry collision mesh filename=package://new_robot/meshes/NONE_1.stl scale=1 1 1; visual mesh filename=package://new_robot/meshes/NONE_1.stl scale=1 1 1
- link none_2: geometry collision mesh filename=package://new_robot/meshes/NONE.stl scale=1 1 1; visual mesh filename=package://new_robot/meshes/NONE.stl scale=1 1 1
- link none_3: geometry collision mesh filename=package://new_robot/meshes/NONE_1.stl scale=1 1 1; visual mesh filename=package://new_robot/meshes/NONE_1.stl scale=1 1 1
- link part_1: geometry collision mesh filename=package://new_robot/meshes/Part_1.stl scale=1 1 1; visual mesh filename=package://new_robot/meshes/Part_1.stl scale=1 1 1
- link part_1_1: geometry collision mesh filename=package://new_robot/meshes/Part_1.stl scale=1 1 1; visual mesh filename=package://new_robot/meshes/Part_1.stl scale=1 1 1
- link part_1_10: geometry collision mesh filename=package://new_robot/meshes/Part_1.stl scale=1 1 1; visual mesh filename=package://new_robot/meshes/Part_1.stl scale=1 1 1
- link part_1_11: geometry collision mesh filename=package://new_robot/meshes/Part_1.stl scale=1 1 1; visual mesh filename=package://new_robot/meshes/Part_1.stl scale=1 1 1
- link part_1_12: geometry collision mesh filename=package://new_robot/meshes/Part_1.stl scale=1 1 1; visual mesh filename=package://new_robot/meshes/Part_1.stl scale=1 1 1
- link part_1_13: geometry collision mesh filename=package://new_robot/meshes/Part_1.stl scale=1 1 1; visual mesh filename=package://new_robot/meshes/Part_1.stl scale=1 1 1
- link part_1_14: geometry collision mesh filename=package://new_robot/meshes/Part_1.stl scale=1 1 1; visual mesh filename=package://new_robot/meshes/Part_1.stl scale=1 1 1
- link part_1_15: geometry collision mesh filename=package://new_robot/meshes/Part_1.stl scale=1 1 1; visual mesh filename=package://new_robot/meshes/Part_1.stl scale=1 1 1
- link part_1_16: geometry collision mesh filename=package://new_robot/meshes/Part_1.stl scale=1 1 1; visual mesh filename=package://new_robot/meshes/Part_1.stl scale=1 1 1
- link part_1_17: geometry collision mesh filename=package://new_robot/meshes/Part_1.stl scale=1 1 1; visual mesh filename=package://new_robot/meshes/Part_1.stl scale=1 1 1
- link part_1_18: geometry collision mesh filename=package://new_robot/meshes/Part_1.stl scale=1 1 1; visual mesh filename=package://new_robot/meshes/Part_1.stl scale=1 1 1
- link part_1_19: geometry collision mesh filename=package://new_robot/meshes/Part_1.stl scale=1 1 1; visual mesh filename=package://new_robot/meshes/Part_1.stl scale=1 1 1
- link part_1_2: geometry collision mesh filename=package://new_robot/meshes/Part_1.stl scale=1 1 1; visual mesh filename=package://new_robot/meshes/Part_1.stl scale=1 1 1
- link part_1_3: geometry collision mesh filename=package://new_robot/meshes/Part_1.stl scale=1 1 1; visual mesh filename=package://new_robot/meshes/Part_1.stl scale=1 1 1
- link part_1_4: geometry collision mesh filename=package://new_robot/meshes/Part_1.stl scale=1 1 1; visual mesh filename=package://new_robot/meshes/Part_1.stl scale=1 1 1
- link part_1_5: geometry collision mesh filename=package://new_robot/meshes/Part_1.stl scale=1 1 1; visual mesh filename=package://new_robot/meshes/Part_1.stl scale=1 1 1
- link part_1_6: geometry collision mesh filename=package://new_robot/meshes/Part_1.stl scale=1 1 1; visual mesh filename=package://new_robot/meshes/Part_1.stl scale=1 1 1
- link part_1_7: geometry collision mesh filename=package://new_robot/meshes/Part_1.stl scale=1 1 1; visual mesh filename=package://new_robot/meshes/Part_1.stl scale=1 1 1
- link part_1_8: geometry collision mesh filename=package://new_robot/meshes/Part_1.stl scale=1 1 1; visual mesh filename=package://new_robot/meshes/Part_1.stl scale=1 1 1
- link part_1_9: geometry collision mesh filename=package://new_robot/meshes/Part_1.stl scale=1 1 1; visual mesh filename=package://new_robot/meshes/Part_1.stl scale=1 1 1
- link Колісний_диск: geometry collision mesh filename=package://new_robot/meshes/_____________.stl scale=1 1 1; visual mesh filename=package://new_robot/meshes/_____________.stl scale=1 1 1
- link Колісний_диск_1: geometry collision mesh filename=package://new_robot/meshes/_____________.stl scale=1 1 1; visual mesh filename=package://new_robot/meshes/_____________.stl scale=1 1 1
- link Колісний_диск_2: geometry collision mesh filename=package://new_robot/meshes/_____________.stl scale=1 1 1; visual mesh filename=package://new_robot/meshes/_____________.stl scale=1 1 1
- link Колісний_диск_3: geometry collision mesh filename=package://new_robot/meshes/_____________.stl scale=1 1 1; visual mesh filename=package://new_robot/meshes/_____________.stl scale=1 1 1
- link Шина700: geometry collision mesh filename=package://new_robot/meshes/____700.stl scale=1 1 1; visual mesh filename=package://new_robot/meshes/____700.stl scale=1 1 1
- link Шина700_1: geometry collision mesh filename=package://new_robot/meshes/____700.stl scale=1 1 1; visual mesh filename=package://new_robot/meshes/____700.stl scale=1 1 1
- link Шина700_2: geometry collision mesh filename=package://new_robot/meshes/____700.stl scale=1 1 1; visual mesh filename=package://new_robot/meshes/____700.stl scale=1 1 1
- link Шина700_3: geometry collision mesh filename=package://new_robot/meshes/____700.stl scale=1 1 1; visual mesh filename=package://new_robot/meshes/____700.stl scale=1 1 1
Joints:
- joint revolute_1: type continuous -> fixed
- joint revolute_2: type continuous -> fixed
- joint revolute_5: axis -0 -0 1 -> 0 0 -1
- joint revolute_6: axis 0 0 -1 -> 0 0 1

Commit message: Update with current state

File: new_robot/urdf/new_robot.urdf (robot description, URDF)
Before this commit: robot new_robot, 69 links, 68 joints
Links:
- added link water_tank, mass 2e-05; collision mesh filename=package://new_robot/meshes/water_tank.stl scale=1 1 1; visual mesh filename=package://new_robot/meshes/water_tank.stl scale=1 1 1
Joints:
- added joint water_tank_joint: type fixed, parent root, child water_tank, origin xyz=-0.515032 0.292627 -0.0950903 rpy=0 -1.5708 0

Commit message: Update with current state

File: new_robot/urdf/new_robot.urdf (robot description, URDF)
Before this commit: robot new_robot, 70 links, 69 joints
Joints:
- joint revolute_1: limit (none) -> lower=-0.4363 upper=0.4363 effort=10 velocity=3.0; type fixed -> revolute
- joint revolute_2: limit (none) -> lower=-0.4363 upper=0.4363 effort=10 velocity=3.0; type fixed -> revolute
- joint water_tank_joint: origin xyz=-0.515032 0.292627 -0.0950903 rpy=0 -1.5708 0 -> xyz=-0.115419 0.019334 0.169057 rpy=0.000498 1.545365 3.080375; parent root -> default_4

Commit message: Update with current state

File: new_robot/urdf/new_robot.urdf (robot description, URDF)
Before this commit: robot new_robot, 70 links, 69 joints
Links:
- link part_1_1: geometry collision cylinder length=0.07 radius=0.105; visual mesh filename=package://new_robot/meshes/Part_1.stl scale=1 1 1
- link part_1_12: geometry collision cylinder length=0.07 radius=0.105; visual mesh filename=package://new_robot/meshes/Part_1.stl scale=1 1 1
- link part_1_13: geometry collision cylinder length=0.07 radius=0.105; visual mesh filename=package://new_robot/meshes/Part_1.stl scale=1 1 1
- link part_1_9: geometry collision cylinder length=0.07 radius=0.105; visual mesh filename=package://new_robot/meshes/Part_1.stl scale=1 1 1
- link water_tank: mass 2e-05 -> 0.5

Commit message: Update with current state

File: new_robot/urdf/new_robot.urdf (robot description, URDF)
Before this commit: robot new_robot, 70 links, 69 joints
Links:
- link body2: mass 0.000770683 -> 0.08
- link body2_1: mass 0.000770683 -> 0.08
- link body2_2: mass 0.000770683 -> 0.08
- link body2_3: mass 0.000770683 -> 0.08
- link part_1: mass 2.44526e-05 -> 0.01
- link part_1_1: mass 2.44526e-05 -> 0.01
- link part_1_10: mass 2.44526e-05 -> 0.01
- link part_1_11: mass 2.44526e-05 -> 0.01
- link part_1_12: mass 2.44526e-05 -> 0.01
- link part_1_13: mass 2.44526e-05 -> 0.01
- link part_1_14: mass 2.44526e-05 -> 0.01
- link part_1_15: mass 2.44526e-05 -> 0.01
- link part_1_16: mass 2.44526e-05 -> 0.01
- link part_1_17: mass 2.44526e-05 -> 0.01
- link part_1_18: mass 2.44526e-05 -> 0.01
- link part_1_19: mass 2.44526e-05 -> 0.01
- link part_1_2: mass 2.44526e-05 -> 0.01
- link part_1_3: mass 2.44526e-05 -> 0.01
- link part_1_4: mass 2.44526e-05 -> 0.01
- link part_1_5: mass 2.44526e-05 -> 0.01
- link part_1_6: mass 2.44526e-05 -> 0.01
- link part_1_7: mass 2.44526e-05 -> 0.01
- link part_1_8: mass 2.44526e-05 -> 0.01
- link part_1_9: mass 2.44526e-05 -> 0.01

Commit message: Update with current state

File: new_robot/urdf/new_robot.urdf (robot description, URDF)
Before this commit: robot new_robot, 70 links, 69 joints
Links:
- link bjj02040274_gl60ii_Å_à_Ç_1_solid1: geometry visual mesh filename=package://new_robot/meshes/BJJ02040274_GL60II_______1_solid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 scale=1 1 1
- link bjj02040274_gl60ii_Å_à_Ç_1_solid1_1: geometry visual mesh filename=package://new_robot/meshes/BJJ02040274_GL60II_______1_solid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 scale=1 1 1
- link body2: geometry collision box size=0.1 0.1 0.06; visual mesh filename=package://new_robot/meshes/Body2.stl scale=1 1 1
- link body2_1: geometry collision box size=0.1 0.1 0.06; visual mesh filename=package://new_robot/meshes/Body2.stl scale=1 1 1
- link body2_2: geometry collision box size=0.1 0.1 0.06; visual mesh filename=package://new_robot/meshes/Body2.stl scale=1 1 1
- link body2_3: geometry collision box size=0.1 0.1 0.06; visual mesh filename=package://new_robot/meshes/Body2.stl scale=1 1 1
- link default: geometry visual mesh filename=package://new_robot/meshes/Default.stl scale=1 1 1
- link default_1: geometry visual mesh filename=package://new_robot/meshes/Default.stl scale=1 1 1
- link default_10: geometry visual mesh filename=package://new_robot/meshes/Default.stl scale=1 1 1
- link default_11: geometry visual mesh filename=package://new_robot/meshes/Default.stl scale=1 1 1
- link default_12: geometry visual mesh filename=package://new_robot/meshes/Default.stl scale=1 1 1
- link default_13: geometry visual mesh filename=package://new_robot/meshes/Default.stl scale=1 1 1
- link default_2: geometry visual mesh filename=package://new_robot/meshes/Default.stl scale=1 1 1
- link default_3: geometry visual mesh filename=package://new_robot/meshes/Default.stl scale=1 1 1
- link default_4: geometry visual mesh filename=package://new_robot/meshes/Default.stl scale=1 1 1
- link default_5: geometry visual mesh filename=package://new_robot/meshes/Default.stl scale=1 1 1
- link default_6: geometry visual mesh filename=package://new_robot/meshes/Default.stl scale=1 1 1
- link default_7: geometry visual mesh filename=package://new_robot/meshes/Default.stl scale=1 1 1
- link default_8: geometry visual mesh filename=package://new_robot/meshes/Default.stl scale=1 1 1
- link default_9: geometry visual mesh filename=package://new_robot/meshes/Default.stl scale=1 1 1
- link gb_fastener_screws_hshcs_m3x5_s_1_solid1: geometry visual mesh filename=package://new_robot/meshes/GB_FASTENER_SCREWS_HSHCS_M3X5_S_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 scale=1 1 1
- link gb_fastener_screws_hshcs_m3x5_s_1_solid1_1: geometry visual mesh filename=package://new_robot/meshes/GB_FASTENER_SCREWS_HSHCS_M3X5_S_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 scale=1 1 1
- link gb_fastener_screws_hshcs_m3x5_s_2_solid1: geometry visual mesh filename=package://new_robot/meshes/GB_FASTENER_SCREWS_HSHCS_M3X5_S_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 scale=1 1 1
- link gb_fastener_screws_hshcs_m3x5_s_2_solid1_1: geometry visual mesh filename=package://new_robot/meshes/GB_FASTENER_SCREWS_HSHCS_M3X5_S_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 scale=1 1 1
- link gb_fastener_screws_hshcs_m3x5_s_4_solid1: geometry visual mesh filename=package://new_robot/meshes/GB_FASTENER_SCREWS_HSHCS_M3X5_S_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 scale=1 1 1
- link gb_fastener_screws_hshcs_m3x5_s_4_solid1_1: geometry visual mesh filename=package://new_robot/meshes/GB_FASTENER_SCREWS_HSHCS_M3X5_S_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 scale=1 1 1
- link gl60_v1_0_240806a_1_solid86: geometry visual mesh filename=package://new_robot/meshes/GL60_V1_0_240806A_1_solid86.stl scale=1 1 1
- link gl60_v1_0_240806a_1_solid86_1: geometry visual mesh filename=package://new_robot/meshes/GL60_V1_0_240806A_1_solid86.stl scale=1 1 1
- link gl60_v1_0_240806a_1_solid87: geometry visual mesh filename=package://new_robot/meshes/GL60_V1_0_240806A_1_solid87.stl scale=1 1 1
- link gl60_v1_0_240806a_1_solid87_1: geometry visual mesh filename=package://new_robot/meshes/GL60_V1_0_240806A_1_solid87.stl scale=1 1 1
- link m3_ÂÝÎÆ__1: geometry visual mesh filename=package://new_robot/meshes/M3_______1.stl scale=1 1 1
- link m3_ÂÝÎÆ__1_1: geometry visual mesh filename=package://new_robot/meshes/M3_______1.stl scale=1 1 1
- link none: geometry visual mesh filename=package://new_robot/meshes/NONE.stl scale=1 1 1
- link none_1: geometry visual mesh filename=package://new_robot/meshes/NONE_1.stl scale=1 1 1
- link none_2: geometry visual mesh filename=package://new_robot/meshes/NONE.stl scale=1 1 1
- link none_3: geometry visual mesh filename=package://new_robot/meshes/NONE_1.stl scale=1 1 1
- link part_1: geometry visual mesh filename=package://new_robot/meshes/Part_1.stl scale=1 1 1
- link part_1_10: geometry visual mesh filename=package://new_robot/meshes/Part_1.stl scale=1 1 1
- link part_1_11: geometry visual mesh filename=package://new_robot/meshes/Part_1.stl scale=1 1 1
- link part_1_14: geometry visual mesh filename=package://new_robot/meshes/Part_1.stl scale=1 1 1
- link part_1_15: geometry visual mesh filename=package://new_robot/meshes/Part_1.stl scale=1 1 1
- link part_1_16: geometry visual mesh filename=package://new_robot/meshes/Part_1.stl scale=1 1 1
- link part_1_17: geometry visual mesh filename=package://new_robot/meshes/Part_1.stl scale=1 1 1
- link part_1_18: geometry visual mesh filename=package://new_robot/meshes/Part_1.stl scale=1 1 1
- link part_1_19: geometry visual mesh filename=package://new_robot/meshes/Part_1.stl scale=1 1 1
- link part_1_2: geometry visual mesh filename=package://new_robot/meshes/Part_1.stl scale=1 1 1
- link part_1_3: geometry visual mesh filename=package://new_robot/meshes/Part_1.stl scale=1 1 1
- link part_1_4: geometry visual mesh filename=package://new_robot/meshes/Part_1.stl scale=1 1 1
- link part_1_5: geometry visual mesh filename=package://new_robot/meshes/Part_1.stl scale=1 1 1
- link part_1_6: geometry visual mesh filename=package://new_robot/meshes/Part_1.stl scale=1 1 1
- link part_1_7: geometry visual mesh filename=package://new_robot/meshes/Part_1.stl scale=1 1 1
- link part_1_8: geometry visual mesh filename=package://new_robot/meshes/Part_1.stl scale=1 1 1
- link water_tank: geometry visual mesh filename=package://new_robot/meshes/water_tank.stl scale=1 1 1
- link Колісний_диск: geometry visual mesh filename=package://new_robot/meshes/_____________.stl scale=1 1 1
- link Колісний_диск_1: geometry visual mesh filename=package://new_robot/meshes/_____________.stl scale=1 1 1
- link Колісний_диск_2: geometry visual mesh filename=package://new_robot/meshes/_____________.stl scale=1 1 1
- link Колісний_диск_3: geometry visual mesh filename=package://new_robot/meshes/_____________.stl scale=1 1 1
- link Шина700: geometry visual mesh filename=package://new_robot/meshes/____700.stl scale=1 1 1
- link Шина700_1: geometry visual mesh filename=package://new_robot/meshes/____700.stl scale=1 1 1
- link Шина700_2: geometry visual mesh filename=package://new_robot/meshes/____700.stl scale=1 1 1
- link Шина700_3: geometry visual mesh filename=package://new_robot/meshes/____700.stl scale=1 1 1
