Commit message: Update with current state

File: new_robot/urdf/new_robot.urdf (robot description, URDF)
Before this commit: robot new_robot, 70 links, 69 joints
Links:
- added link slosh_bob, mass 0.1654; visual sphere radius=0.012
- added link slosh_gimbal_x, mass 0.005
- link water_tank: mass 0.5 -> 0.6899
Joints:
- added joint slosh_pendulum_x: type revolute, parent water_tank, child slosh_gimbal_x, origin xyz=0 0 0.00294 rpy=0 0 0, axis 1 0 0, limit lower=-0.6 upper=0.6 effort=1.0 velocity=20.0
- added joint slosh_pendulum_y: type revolute, parent slosh_gimbal_x, child slosh_bob, origin xyz=0 0 -0.03002 rpy=0 0 0, axis 0 1 0, limit lower=-0.6 upper=0.6 effort=1.0 velocity=20.0
- joint revolute_1: limit lower=-0.4363 upper=0.4363 effort=10 velocity=3.0 -> lower=-0.4363 upper=0.4363 effort=2.5 velocity=3.0
- joint revolute_2: limit lower=-0.4363 upper=0.4363 effort=10 velocity=3.0 -> lower=-0.4363 upper=0.4363 effort=2.5 velocity=3.0
